File: docs/PCB/Boards/Regulator_Board/Regulator_Board.kicad_sch (KiCad schematic)
At the start: 28 parts, among them U1 LM2596S-5, U2 LM2596S-5, U3 LM2596S-5

Commit message: Hardware docs updated.
Parts:
- removed C10: 120uF, symbol Device:C_Polarized
- removed C11, C13, C4, C6, C8: 100nF, symbol Device:C
- removed C12, C3: 330uF, symbol Device:C_Polarized
- removed C5: 180uF, symbol Device:C_Polarized
- removed C7: 470uF, symbol Device:C_Polarized
- removed C9: 1.2nF, symbol Device:C
- removed D2, D3: 1N5822, symbol Device:D_Schottky
- removed L2, L3: 33uH, symbol Device:L
- removed U2, U3: LM2596S-5, Package_TO_SOT_SMD:TO-263-5_TabPin3, symbol Regulator_Switching:LM2596S-5
- added C3: 1.2nF, symbol Device:C
- added C4: 330uF, symbol Device:C_Polarized
- added C5: 100nF, symbol Device:C
- added J1: Jack-DC, Connector_BarrelJack:BarrelJack_Horizontal, symbol Connector:Jack-DC
- added J2: PWR, TerminalBlock_Phoenix:TerminalBlock_Phoenix_MKDS-1,5-2_1x02_P5.00mm_Horizontal, symbol Connector:Screw_Terminal_01x02
- C1: value 120uF -> 330uF
- D1: value 1N5822 -> 1N5825
- R1: value 1KR -> 1K
- R2: value 3K09R -> 3K09
- U1: value LM2596S-5 -> LM2596-5
Connections:
- net +5V: now also C4.1, C5.1, J2.1 (Pin_1); no longer R2.2
- net +VDC: now also J1.1
- net GND: now also C4.2, C5.2, J1.2, J2.2 (Pin_2)
- net at R1.2, R2.1: now also C3.1
- new net: C3.2, R2.2
