File: docs/PCB/Boards/ATMegaSMD_Board/ATMegaSMD_Board.kicad_pcb (KiCad board)
At the start: 2 copper layers, 71.7 x 50.2 mm, 21 parts, among them J1 Conn_02x12_Odd_Even, J2 AVR-ISP-10, J3 Conn_01x10_Pin, J4 Conn_01x10_Pin, SW1 Tact Switch 6x6mm / 13mm, U1 ATmega328PB-A, Y1 Crystal

Commit message: Code review
Parts:
- added D1: LED_SCK, LED_SMD:LED_0805_2012Metric, F.Cu at (180.0, 108.5)
- added D3: LED_PWR, LED_SMD:LED_0805_2012Metric, F.Cu at (189.5, 79.5)
- added Q1: BC847, Package_TO_SOT_SMD:SOT-23, F.Cu at (184.1, 107.8)
- added R2: 1K, Resistor_SMD:R_0805_2012Metric, F.Cu at (189.5, 81.5)
- added R3: 10kR, Resistor_SMD:R_0805_2012Metric, F.Cu at (183.7, 105.0)
- added R4: 1K, Resistor_SMD:R_0805_2012Metric, F.Cu at (180.0, 106.6)
- moved L1 2.49 mm to (140.2, 110.2)
- moved C1 1.38 mm to (140.1, 104.4)
- moved C3 1.31 mm to (140.3, 91.5)
- moved C5 1.23 mm to (140.1, 108.4)
- moved C6 0.76 mm to (139.8, 97.2)
- moved C8 0.56 mm to (139.8, 99.2)
Routing:
- net VCC: track 154.0 -> 169.9 mm, vias 2 -> 3
- net Net-(D1-K): track 0.00 -> 11.5 mm
- net PB5: track 47.3 -> 57.8 mm
- net AVCC: track 50.1 -> 47.6 mm
- net Net-(D3-A): track 0.00 -> 2.02 mm
- net Net-(D1-A): track 0.00 -> 1.97 mm
- net Net-(Q1-B): track 0.00 -> 1.94 mm
- net XTAL1: track 13.4 -> 14.2 mm
- net AREF: track 43.8 -> 43.2 mm

Commit message: Boards modified.
Parts:
- added R5: 100kR, Resistor_SMD:R_0805_2012Metric, F.Cu at (189.0, 105.0)
- J1: footprint Connector_PinHeader_2.00mm:PinHeader_2x12_P2.00mm_Vertical -> Connector_PinHeader_2.54mm:PinHeader_2x12_P2.54mm_Vertical
- R1: value 1K -> 10kR
- Y1: value Crystal -> 16MHz
- moved J1 0.72 mm to (171.8, 78.8)
- moved D1 0.14 mm to (180.2, 108.5)
- moved R4 0.14 mm to (180.2, 106.6)
Routing:
- net PD5: track 41.1 -> 48.5 mm
- net PB3: track 49.9 -> 56.6 mm
- net PB5: track 57.8 -> 64.4 mm
- net Net-(Q1-B): track 1.94 -> 8.06 mm
- net PD6: track 37.3 -> 43.2 mm
- net PB0: track 27.1 -> 32.7 mm
- net PB4: track 53.2 -> 58.7 mm
- net PD7: track 32.4 -> 37.8 mm
- net VCC: track 169.9 -> 174.1 mm
- net PB1: track 21.2 -> 25.0 mm
- net PB2: track 17.2 -> 19.2 mm
- net PE1: track 63.5 -> 65.5 mm
- net PE0: track 55.9 -> 57.5 mm
- net PD4: track 50.6 -> 51.6 mm
- net PD0: track 26.7 -> 25.9 mm
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