File: docs/PCB/Boards/ATMegaSMD_Board/ATMegaSMD_Board.kicad_sch (KiCad schematic)
At the start: 17 parts, among them J17 AVR-ISP-10, J18 Conn_02x10_Odd_Even, J19 Conn_01x10_Pin, J20 Conn_01x10_Pin, SW2 Tact Switch 6x6mm / 13mm, U2 ATmega328P-P, Y4 Crystal

Commit message: Hardware docs updated.
Parts:
- removed J18: Conn_02x10_Odd_Even, Connector_PinHeader_2.54mm:PinHeader_2x10_P2.54mm_Vertical, symbol Connector_Generic:Conn_02x10_Odd_Even
- removed J19: Conn_01x10_Pin, Connector_PinHeader_2.54mm:PinHeader_1x10_P2.54mm_Vertical, symbol Connector:Conn_01x10_Pin
- removed U2: ATmega328P-P, Package_DIP:DIP-28_W7.62mm, symbol MCU_Microchip_ATmega:ATmega328P-P
- added H1, H2, H3, H4: MountingHole_Pad, MountingHole:MountingHole_3.2mm_M3_DIN965_Pad, symbol Mechanical:MountingHole_Pad
- added J1: Conn_02x12_Odd_Even, Connector_PinHeader_2.00mm:PinHeader_2x12_P2.00mm_Vertical, symbol Connector_Generic:Conn_02x12_Odd_Even
- added J3: Conn_01x10_Pin, Connector_PinHeader_2.54mm:PinHeader_1x10_P2.54mm_Vertical, symbol Connector:Conn_01x10_Pin
- added U1: ATmega328PB-A, Package_QFP:TQFP-32_7x7mm_P0.8mm, symbol MCU_Microchip_ATmega:ATmega328PB-A
- renumbered C13 to C1, C14 to C2, C15 to C3, C16 to C4, C17 to C5, C18 to C6, C19 to C7, C20 to C8, J17 to J2, J20 to J4, L6 to L1, R37 to R1, SW2 to SW1, Y4 to Y1
Connections:
- net 5V: now also J3.1 (Pin_1), J3.10 (Pin_10), J3.2 (Pin_2), J3.3 (Pin_3), J3.4 (Pin_4), J3.5 (Pin_5), J3.6 (Pin_6), J3.7 (Pin_7), J3.8 (Pin_8), J3.9 (Pin_9), U1.4 (VCC)
- net GND: now also H1.1, H2.1, H3.1, H4.1, U1.21 (GND), U1.5 (GND)
- net PB0: now also J1.22 (Pin_22), U1.12 (PB0)
- net PB1: now also J1.24 (Pin_24), U1.13 (PB1)
- net PB2: now also J1.23 (Pin_23), U1.14 (PB2)
- net PB3: now also J1.21 (Pin_21), U1.15 (PB3)
- net PB4: now also J1.19 (Pin_19), U1.16 (PB4)
- net PB5: now also J1.17 (Pin_17), U1.17 (PB5)
- net PC0: now also J1.11 (Pin_11), U1.23 (PC0)
- net PC1: now also J1.9 (Pin_9), U1.24 (PC1)
- net PC2: now also J1.7 (Pin_7), U1.25 (PC2)
- net PC3: now also J1.5 (Pin_5), U1.26 (PC3)
- net PC4: now also J1.3 (Pin_3), U1.27 (PC4)
- net PC5: now also J1.1 (Pin_1), U1.28 (PC5)
- net PD0: now also J1.2 (Pin_2), U1.30 (PD0)
- net PD1: now also J1.4 (Pin_4), U1.31 (PD1)
- net PD2: now also J1.6 (Pin_6), U1.32 (PD2)
- net PD3: now also J1.8 (Pin_8), U1.1 (PD3)
- net PD4: now also J1.10 (Pin_10), U1.2 (PD4)
- net PD5: now also J1.16 (Pin_16), U1.9 (PD5)
- net PD6: now also J1.18 (Pin_18), U1.10 (PD6)
- net PD7: now also J1.20 (Pin_20), U1.11 (PD7)
- net RESET: now also U1.29 (~{RESET}/PC6)
- net AREF: now reaches C1.2
- net AREF: now also U1.20 (AREF)
- net XTAL1: now reaches C6.1
- net XTAL1: now also U1.7 (XTAL1/PB6)
- net AVCC: now reaches C4.1, C5.1, L1.2
- net AVCC: now also U1.18 (AVCC)
- net XTAL2: now reaches C8.2
- net XTAL2: now also U1.8 (XTAL2/PB7)
- new net PE0: J1.12 (Pin_12), U1.3 (PE0)
- new net PE1: J1.14 (Pin_14), U1.6 (PE1)
- new net PE2: J1.15 (Pin_15), U1.19 (PE2)
- new net PE3: J1.13 (Pin_13), U1.22 (PE3)
Other:
- title: ATMega328 -> CAN_Board
- moved on the sheet: C1, C2, C3, C4, C5, C6, C7, C8, J2, J4, L1, R1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

Commit message: Boards modified - tree and power boards added.
Other:
- title: CAN_Board -> ATMegaSMD_Board
Changed lines of the file:
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@@
 	(paper "A4")
 	(title_block
-		(title "CAN_Board")
+		(title "ATMegaSMD_Board")
 		(date "2025-10-26")
 		(rev "1.0")

Commit message: Code review
Parts:
- added D1: LED_SCK, LED_SMD:LED_0805_2012Metric, symbol Device:LED
- added D3: LED_PWR, LED_SMD:LED_0805_2012Metric, symbol Device:LED
- added Q1: BC847, Package_TO_SOT_SMD:SOT-23, symbol Transistor_BJT:BC847
- added R2, R4: 1K, Resistor_SMD:R_0805_2012Metric, symbol Device:R
- added R3: 10kR, Resistor_SMD:R_0805_2012Metric, symbol Device:R
Connections:
- net 5V: now also R2.2, R4.2
- net GND: now also D3.1 (K), Q1.2 (E)
- net PB5: now also R3.2
- new net: Q1.1 (B), R3.1
- new net: D3.2 (A), R2.1
- new net: D1.1 (K), Q1.3 (C)
- new net: D1.2 (A), R4.1

Commit message: Boards modified.
Parts:
- added R5: 100kR, Resistor_SMD:R_0805_2012Metric, symbol Device:R
- J1: footprint Connector_PinHeader_2.00mm:PinHeader_2x12_P2.00mm_Vertical -> Connector_PinHeader_2.54mm:PinHeader_2x12_P2.54mm_Vertical
- R1: value 1K -> 10kR
- Y1: value Crystal -> 16MHz
Connections:
- net GND: now also R5.1
- net at Q1.1 (B), R3.1: now also R5.2
Other:
- moved on the sheet: C2, C4, C6, C8, L1, Y1
