File: docs/PCB/Boards/ATMega_Board/ATMega_Board.kicad_pcb (KiCad board)
At the start: 2 copper layers, 128 x 74.8 mm, 21 parts, among them J1 Conn_02x10_Odd_Even, J2 AVR-ISP-10, J3 Conn_01x10_Pin, J4 Conn_01x10_Pin, SW1 Tact Switch 6x6mm / 13mm, U2 ATmega328P-P, Y1 Crystal

Commit message: Hardware docs updated.
Parts:
- moved H4 58.1 mm to (190.0, 115.0)
- moved H1 57.5 mm to (190.0, 72.0)
- moved H3 13.9 mm to (125.1, 115.0)
- moved H2 11.0 mm to (125.1, 72.0)
Other:
- board size 128 x 74.8 mm -> 71.7 x 50.2 mm
Changed lines of the file:
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@@
 		(tags "Through hole pin header THT 1x10 2.54mm single row")
 		(property "Reference" "J4"
-			(at 0 25.355 0)
+			(at 0 -2.345 0)
 			(layer "F.SilkS")
 			(effects
@@
 	(footprint "MountingHole:MountingHole_3.2mm_M3_DIN965_Pad"
 		(layer "F.Cu")
-		(at 125.05 61.05)
+		(at 125.1 72)
 		(descr "Mounting Hole 3.2mm, M3, generated by kicad-footprint-generator mountinghole.py")
 		(tags "mountinghole M3 DIN965")
@@
 		(tags "Through hole pin header THT 1x10 2.54mm single row")
 		(property "Reference" "J3"
-			(at 0 25.31 0)
+			(at 0 -2.39 0)
 			(layer "F.SilkS")
 			(effects
@@
 	(footprint "MountingHole:MountingHole_3.2mm_M3_DIN965_Pad"
 		(layer "F.Cu")
-		(at 125.05 128.85)
+		(at 125.1 115)
 		(descr "Mounting Hole 3.2mm, M3, generated by kicad-footprint-generator mountinghole.py")
 		(tags "mountinghole M3 DIN965")
@@
 	(footprint "MountingHole:MountingHole_3.2mm_M3_DIN965_Pad"
 		(layer "F.Cu")
-		(at 246.45 128.7)
+		(at 190 115)
 		(descr "Mounting Hole 3.2mm, M3, generated by kicad-footprint-generator mountinghole.py")
 		(tags "mountinghole M3 DIN965")
@@
 	(footprint "MountingHole:MountingHole_3.2mm_M3_DIN965_Pad"
 		(layer "F.Cu")
-		(at 246.45 61.05)
+		(at 190 72)
 		(descr "Mounting Hole 3.2mm, M3, generated by kicad-footprint-generator mountinghole.py")
 		(tags "mountinghole M3 DIN965")
@@
 	)
 	(gr_rect
-		(start 227.925 128.85)
-		(end 242.225 130.85)
+		(start 171.95 114.8)
+		(end 186.25 116.8)
 		(stroke
 			(width 0.15)
@@
 	)
 	(gr_rect
-		(start 121.707152 57.44)
-		(end 249.75 132.195)
+		(start 121.707152 68.44)
+		(end 193.45 118.595)
 		(stroke
 			(width 0.05)
@@
 	)
 	(gr_text "ATMega Board 1.0"
-		(at 228.1 130.35 0)
+		(at 172.125 116.3 0)
 		(layer "F.SilkS")
 		(effects
@@
 		(polygon
 			(pts
-				(xy 249.75 57.45) (xy 249.75 132.2) (xy 121.7 132.2) (xy 121.7 57.45)
+				(xy 193.45 68.45) (xy 193.45 118.59) (xy 121.71 118.59) (xy 121.7 68.45)
 			)
 		)

Commit message: Code review
Parts:
- added D1: LED_SCK, LED_SMD:LED_0805_2012Metric, F.Cu at (177.0, 107.5)
- added D3: LED_PWR, LED_SMD:LED_0805_2012Metric, F.Cu at (178.9, 80.5)
- added Q1: BC847, Package_TO_SOT_SMD:SOT-23, F.Cu at (177.0, 104.7)
- added R2: 1K, Resistor_SMD:R_0805_2012Metric, F.Cu at (179.0, 82.5)
- added R3: 10kR, Resistor_SMD:R_0805_2012Metric, F.Cu at (176.7, 102.0)
- added R4: 1K, Resistor_SMD:R_0805_2012Metric, F.Cu at (177.0, 109.5)
- moved L1 2.52 mm to (161.3, 101.8)
- moved C6 1.66 mm to (146.5, 97.1)
- moved C8 1.61 mm to (146.5, 99.7)
- moved C3 1.29 mm to (145.2, 91.6)
- moved C5 1.23 mm to (161.3, 100.0)
Routing:
- net VCC: track 129.5 -> 143.8 mm
- net PB5: track 51.6 -> 56.1 mm
- net PB4: track 42.7 -> 45.9 mm
- net Net-(D1-K): track 0.00 -> 2.84 mm
- net AVCC: track 10.0 -> 7.46 mm
- net Net-(D3-A): track 0.00 -> 2.07 mm
- net Net-(D1-A): track 0.00 -> 2.00 mm
- net Net-(Q1-B): track 0.00 -> 1.99 mm
- net XTAL2: track 3.79 -> 1.95 mm
- net Net-(C6-Pad2): track 4.23 -> 6.02 mm
- net XTAL1: track 3.72 -> 1.97 mm
- net Net-(C8-Pad1): track 4.41 -> 6.15 mm
- net GND: vias 1 -> 2

Commit message: Boards modified.
Parts:
- added R5: 100kR, Resistor_SMD:R_0805_2012Metric, F.Cu at (180.7, 106.0)
- R1: value 1K -> 10kR
- Y1: value Crystal -> 16MHz
Routing:
- net Net-(Q1-B): track 1.99 -> 7.83 mm
