File: docs/PCB/Boards/ATMega_Board/ATMega_Board.kicad_sch (KiCad schematic)
At the start: 22 parts, among them J1 Conn_02x10_Odd_Even, J2 AVR-ISP-10, J3 Conn_01x10_Pin, J4 Conn_01x10_Pin, SW1 Tact Switch 6x6mm / 13mm, U1 ATmega328PB-A, U2 ATmega328P-P, Y1 Crystal

Commit message: Hardware docs updated.
Parts:
- removed U1: ATmega328PB-A, Package_QFP:TQFP-32_7x7mm_P0.8mm, symbol MCU_Microchip_ATmega:ATmega328PB-A
Other:
- moved on the sheet: J1, J2, J3, J4

Commit message: Boards modified - tree and power boards added.
Other:
- title: CAN_Board -> ATMega_Board
Changed lines of the file:
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@@
 	(paper "A4")
 	(title_block
-		(title "CAN_Board")
+		(title "ATMega_Board")
 		(date "2025-10-26")
 		(rev "1.0")

Commit message: Code review
Parts:
- added D1: LED_SCK, LED_SMD:LED_0805_2012Metric, symbol Device:LED
- added D3: LED_PWR, LED_SMD:LED_0805_2012Metric, symbol Device:LED
- added Q1: BC847, Package_TO_SOT_SMD:SOT-23, symbol Transistor_BJT:BC847
- added R2, R4: 1K, Resistor_SMD:R_0805_2012Metric, symbol Device:R
- added R3: 10kR, Resistor_SMD:R_0805_2012Metric, symbol Device:R
Connections:
- net 5V: now also R2.2, R4.2
- net GND: now also D3.1 (K), Q1.2 (E)
- net PB5: now also R3.2
- new net: Q1.1 (B), R3.1
- new net: D3.2 (A), R2.1
- new net: D1.1 (K), Q1.3 (C)
- new net: D1.2 (A), R4.1

Commit message: Boards modified.
Parts:
- added R5: 100kR, Resistor_SMD:R_0805_2012Metric, symbol Device:R
- R1: value 1K -> 10kR
- Y1: value Crystal -> 16MHz
Connections:
- net GND: now also R5.2
- net at Q1.1 (B), R3.1: now also R5.1
Other:
- moved on the sheet: C1, C2, C3, C4, C6, C8, L1, Y1
