File: docs/PCB/Boards/CAN_Board/CAN_Board.kicad_sch (KiCad schematic)
At the start: 30 parts, among them J1 COM, J2 CAN, Q1 AO3407A, U1 MCP2515-I/SO, U2 SN65HVD230DR, U3 SIP32431DR3-T1GE3, Y1 3225-20M-SR

Commit message: Boards modified.
Parts:
- R6: value 1K -> 4k7R
Changed lines of the file:
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@@
 			)
 		)
-		(property "Value" "1K"
+		(property "Value" "4k7R"
 			(at 201.93 113.03 90)
 			(effects
