File: docs/PCB/Boards/EEPROM_Board/EEPROM_Board.kicad_sch (KiCad schematic)
At the start: 20 parts, among them J1 COM, Q1 AO3407A, SW1 SW_DIP_x04, U1 M24C32-WMN6TP, U2 SIP32431DR3-T1GE3

Commit message: Boards modified.
Parts:
- R7: value 1K -> 4k7R
Changed lines of the file:
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@@
 			)
 		)
-		(property "Value" "1K"
+		(property "Value" "4k7R"
 			(at 165.1 106.68 90)
 			(effects
