File: docs/PCB/Boards/GPIO_Board/GPIO_Board.kicad_sch (KiCad schematic)
At the start: 25 parts, among them J1 COM, J2 GPIO, Q1 AO3407A, SW1 SW_DIP_x03, SW2 Tact Switch 6x6mm / 13mm, U1 MCP23017_SS, U2 SIP32431DR3-T1GE3

Commit message: Boards modified.
Parts:
- R7: value 1K -> 4k7R
Changed lines of the file:
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@@
 			)
 		)
-		(property "Value" "1K"
+		(property "Value" "4k7R"
 			(at 162.56 115.57 90)
 			(effects
