File: docs/PCB/Boards/MOSFET_Board/1.0/MOSFET_Board.kicad_pcb (KiCad board)
At the start: 2 copper layers, 57.8 x 26.3 mm, 19 parts, among them IC1 TC4420EOA, J1 COM, J2 BULB, J3 PWR, Q1 AOD4184A

Commit message: Boards modified.
Parts:
- removed D2: SS54BF-DC, Diode_SMD:D_SMB
- removed D3: SMBJ18A-LF, Diode_SMD:D_SMB
- added C1: 330nF, Capacitor_SMD:C_1206_3216Metric, F.Cu at (139.1, 78.3)
- added C4: 100nF, Capacitor_SMD:C_1206_3216Metric, F.Cu at (132.2, 82.8)
- added U1: L78L12ABUTR, Package_TO_SOT_SMD:SOT-89-3, F.Cu at (138.9, 73.0)
- moved C2 14.9 mm to (144.1, 73.7), turned to 0 degrees
- moved D1 4.27 mm to (145.9, 77.6)
- moved R4 2.97 mm to (145.9, 81.3)
- moved IC1 2.66 mm to (139.8, 82.4)
- moved R3 1.94 mm to (145.9, 84.9)
Connections:
- net +12V_SEC renamed +12V_STAB
Routing:
- net +12V: track 19.8 -> 27.2 mm, vias 12 -> 4
- net +12V_STAB: track 24.8 -> 28.5 mm
- net Net-(IC1-INPUT): track 7.56 -> 10.1 mm
- net Net-(D1-K): track 3.93 -> 4.93 mm
- net Net-(IC1-OUTPUT_1): track 3.59 -> 4.58 mm
- net Net-(Q1-G): track 7.72 -> 7.12 mm
- net GND: vias 41 -> 40
Other:
- board text added: "MOSFET Board 1.0"
- board text removed: "MOSFET Board 1.1"
