File: docs/PCB/Boards/MOSFET_Board/1.0/MOSFET_Board.kicad_sch (KiCad schematic)
At the start: 15 parts, among them IC1 TC4420EOA, J1 COM, J2 BULB, J3 PWR, Q1 AOD4184A

Commit message: Boards modified.
Parts:
- removed D2: SS54BF-DC, Diode_SMD:D_SMB, symbol Diode:B230
- removed D3: SMBJ18A-LF, Diode_SMD:D_SMB, symbol Diode:SM6T6V8A
- added C1: 330nF, Capacitor_SMD:C_1206_3216Metric, symbol Device:C_Small
- added C4: 100nF, Capacitor_SMD:C_1206_3216Metric, symbol Device:C_Small
- added U1: L78L12ABUTR, Package_TO_SOT_SMD:SOT-89-3, symbol Regulator_Linear:L78L12_SOT89
Connections:
- net +12V: now also C1.1, U1.3 (IN)
- net GND: now also C1.2, C4.2, U1.2 (GND)
- net +12V_SEC renamed +12V_STAB
- net +12V_STAB: now also C4.1, U1.1 (OUT)
