File: docs/PCB/Boards/Modbus_Board/Modbus_Board.kicad_sch (KiCad schematic)
At the start: 20 parts, among them J1 Modbus, J12 COM, Q1 AO3407A, U1 MAX3485CSA+, U2 SIP32431DR3-T1GE3

Commit message: Boards modified.
Parts:
- R4: value 1K -> 4k7R
Changed lines of the file:
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@@
 			)
 		)
-		(property "Value" "1K"
+		(property "Value" "4k7R"
 			(at 163.83 125.73 90)
 			(effects
