File: docs/PCB/Boards/Power_Board/Power_Board.kicad_pcb (KiCad board)
At the start: 2 copper layers, 71.7 x 45.6 mm, 30 parts, among them J1 IN, J2 12V1, J3 12V2, J4 9V1, J5 9V2, J6 3V3, J7 3V_GND, J8 5V, J9 5V_GND, U1 L7809, U3 AMS1117-3.3, U4 AP63200WU

Commit message: Boards modified.
Parts:
- removed U4: AP63200WU, Package_TO_SOT_SMD:TSOT-23-6
- added C12: 22uF, Capacitor_SMD:C_1206_3216Metric, F.Cu at (164.3, 100.7)
- added C13: 22uF, Capacitor_SMD:C_1206_3216Metric, F.Cu at (148.2, 105.0)
- added C14: 100nF, Capacitor_SMD:C_1206_3216Metric, F.Cu at (148.2, 102.7)
- added C15: 100nF, Capacitor_SMD:C_0805_2012Metric, F.Cu at (142.8, 109.5)
- added C16: 100pF, Capacitor_SMD:C_0805_2012Metric, F.Cu at (146.3, 110.3)
- added C17: 22uF, Capacitor_SMD:C_1206_3216Metric, F.Cu at (143.4, 98.5)
- added C18: 22uF, Capacitor_SMD:C_1206_3216Metric, F.Cu at (143.4, 100.8)
- added L1: DR127-100-R, Inductor_SMD:L_12x12mm_H8mm, F.Cu at (158.2, 90.3)
- added L3: DR73-6R8-R, Inductor_SMD:L_7.3x7.3_H3.5, F.Cu at (136.8, 106.0)
- added R3: 158kR, Resistor_SMD:R_0805_2012Metric, F.Cu at (167.2, 112.2)
- added R4: 30kR, Resistor_SMD:R_0805_2012Metric, F.Cu at (167.2, 108.2)
- added R5: 182kR, Resistor_SMD:R_0805_2012Metric, F.Cu at (146.3, 112.3)
- added R6: 62kR, Resistor_SMD:R_0805_2012Metric, F.Cu at (146.3, 108.3)
- added U2: AP63200WU, Package_TO_SOT_SMD:TSOT-23-6, F.Cu at (164.2, 105.2)
- C1: value 330nF -> 22uF; footprint Capacitor_SMD:C_0805_2012Metric -> Capacitor_SMD:C_1206_3216Metric
- C10: value 10uF -> 100pF
- C11: value 100nF -> 22uF; footprint Capacitor_SMD:C_0805_2012Metric -> Capacitor_SMD:C_1206_3216Metric
- C2: footprint Capacitor_SMD:C_0805_2012Metric -> Capacitor_SMD:C_1206_3216Metric
- C3: value 10uF -> 100nF; footprint Capacitor_SMD:C_1206_3216Metric -> Capacitor_SMD:C_0805_2012Metric
- C4: value 100nF -> 68pF
- C5: value 100pF -> 22uF; footprint Capacitor_SMD:C_0805_2012Metric -> Capacitor_SMD:C_1206_3216Metric
- C8: value 10uF -> 100nF; footprint Capacitor_SMD:C_0805_2012Metric -> Capacitor_SMD:C_1206_3216Metric
- L2: value DE1207-10 -> DR73-100-R; footprint Inductor_SMD:L_12x12mm_H8mm -> Inductor_SMD:L_7.3x7.3_H3.5
- R1: value 157kR -> 182kR
- R2: value 30kR -> 18kR
- U1: value L7809 -> AP63200WU; footprint Package_TO_SOT_SMD:TO-263-2 -> Package_TO_SOT_SMD:TSOT-23-6
- U3: value AMS1117-3.3 -> AP63200WU; footprint Package_TO_SOT_SMD:SOT-223-3_TabPin2 -> Package_TO_SOT_SMD:TSOT-23-6
- moved C10 30.9 mm to (167.2, 110.2), turned to 0 degrees
- moved C5 26.5 mm to (167.4, 82.2), turned to 0 degrees
- moved J9 25.2 mm to (145.9, 78.5)
- moved C11 20.7 mm to (164.3, 98.3), turned to 0 degrees
- moved R2 20.3 mm to (170.3, 92.7), turned to 0 degrees
- moved C4 20.0 mm to (170.3, 94.7)
- moved C8 19.2 mm to (169.2, 102.5)
- moved C9 18.8 mm to (163.7, 109.3)
- moved C6 18.1 mm to (167.4, 85.3)
- moved U3 17.7 mm to (143.3, 105.4), turned to 180 degrees
- moved R1 14.9 mm to (170.3, 96.7), turned to 0 degrees
- moved J8 13.9 mm to (145.9, 87.8)
- moved C7 13.6 mm to (169.2, 104.8)
- moved L2 11.2 mm to (157.7, 105.9)
- moved C3 10.5 mm to (166.8, 93.9), turned to 0 degrees
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Connections:
- C10 pad 1: 3V3 -> 5V
- C10 pad 2: GND -> Net-(U2-FB)
- C11 pad 1: 3V3 -> 5V
- C11 pad 2: GND -> Net-(C11-Pad2)
- C2 pad 1: 9V -> 12V
- C3 pad 1: 12V -> Net-(U1-SW)
- C3 pad 2: GND -> Net-(U1-BST)
- C4 pad 1: Net-(U4-SW) -> 9V
- C4 pad 2: Net-(U4-BST) -> Net-(U1-FB)
- C5 pad 1: 5V -> 9V
- C5 pad 2: Net-(U4-FB) -> Net-(C5-Pad2)
- C6 pad 1: 5V -> Net-(C5-Pad2)
- C6 pad 2: Net-(C6-Pad2) -> GND
- C7 pad 1: Net-(C6-Pad2) -> 12V
- C8 pad 1: 5V -> 12V
- C9 pad 1: 5V -> Net-(U2-SW)
- C9 pad 2: GND -> Net-(U2-BST)
- L2 pad 1: Net-(U4-SW) -> Net-(U2-SW)
- R1 pad 1: 5V -> 9V
- R1 pad 2: Net-(U4-FB) -> Net-(U1-FB)
- R2 pad 1: Net-(U4-FB) -> Net-(U1-FB)
- U1 pad 1: 12V -> Net-(U1-FB)
- U1 pad 2: GND -> 12V
- U1 pad 3: 9V -> 12V
- U3 pad 1: GND -> Net-(U3-FB)
- U3 pad 2: 3V3 -> 12V
- U3 pad 3: 5V -> 12V
Routing:
- net 5V: track 66.4 -> 17.0 mm, vias 2 -> 20
- net 3V3: track 34.6 -> 17.0 mm, vias 0 -> 18
- net 9V: track 3.83 -> 17.8 mm, vias 16 -> 35
- net 12V: track 37.1 -> 45.7 mm, vias 15 -> 40
- net Net-(U4-FB): track 8.38 -> 0.00 mm
- net Net-(U2-FB): track 0.00 -> 7.98 mm
- net Net-(U3-FB): track 0.00 -> 7.51 mm
- net Net-(U1-FB): track 0.00 -> 7.19 mm
- net Net-(C5-Pad2): track 0.00 -> 4.67 mm
- net Net-(C6-Pad2): track 4.66 -> 0.00 mm
- net Net-(U2-BST): track 0.00 -> 4.18 mm
- net Net-(U3-BST): track 0.00 -> 4.07 mm
- net Net-(U1-BST): track 0.00 -> 4.06 mm
- net Net-(C11-Pad2): track 0.00 -> 3.92 mm
- net Net-(C17-Pad2): track 0.00 -> 3.92 mm
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- added copper zone on B.Cu, net (none)
- added copper zone on F.Cu, net Net-(U1-SW)
- added copper zone on F.Cu, net Net-(U2-SW)
- added copper zone on F.Cu, net Net-(U3-SW)
- removed copper zone on F.Cu, net Net-(U4-SW)
Other:
- board text added: "Power Board 1.1"
- board text removed: "Power Board 1.0"
