File: docs/PCB/Boards/Power_Board/1.0/Power_Board.kicad_sch (KiCad schematic)
At the start: 43 parts, among them J1 IN, J2 12V1, J3 12V2, J4 9V1, J5 9V2, J6 3V3, J7 3V_GND, J8 5V, J9 5V_GND, U1 AP63200WU, U2 AP63200WU, U3 AP63200WU

Commit message: Boards modified.
Parts:
- removed C12, C13, C17, C18: 22uF, Capacitor_SMD:C_1206_3216Metric, symbol Device:C
- removed C14: 100nF, Capacitor_SMD:C_1206_3216Metric, symbol Device:C
- removed C15: 100nF, Capacitor_SMD:C_0805_2012Metric, symbol Device:C
- removed C16: 100pF, Capacitor_SMD:C_0805_2012Metric, symbol Device:C
- removed L1: DR127-100-R, Inductor_SMD:L_12x12mm_H8mm, symbol Device:L
- removed L3: DR73-6R8-R, Inductor_SMD:L_7.3x7.3_H3.5, symbol Device:L
- removed R3: 158kR, Resistor_SMD:R_0805_2012Metric, symbol Device:R
- removed R4: 30kR, Resistor_SMD:R_0805_2012Metric, symbol Device:R
- removed R5: 182kR, Resistor_SMD:R_0805_2012Metric, symbol Device:R
- removed R6: 62kR, Resistor_SMD:R_0805_2012Metric, symbol Device:R
- removed U1, U2, U3: AP63200WU, Package_TO_SOT_SMD:TSOT-23-6, symbol Regulator_Switching:AP63200WU
- added U1: L7809, Package_TO_SOT_SMD:TO-263-2, symbol Regulator_Linear:L7809
- added U3: AMS1117-3.3, Package_TO_SOT_SMD:SOT-223-3_TabPin2, symbol Regulator_Linear:AMS1117-3.3
- added U4: AP63200WU, Package_TO_SOT_SMD:TSOT-23-6, symbol Regulator_Switching:AP63200WU
- C1: value 22uF -> 330nF; footprint Capacitor_SMD:C_1206_3216Metric -> Capacitor_SMD:C_0805_2012Metric
- C10: value 100pF -> 10uF
- C11: value 22uF -> 100nF; footprint Capacitor_SMD:C_1206_3216Metric -> Capacitor_SMD:C_0805_2012Metric
- C2: footprint Capacitor_SMD:C_1206_3216Metric -> Capacitor_SMD:C_0805_2012Metric
- C3: value 100nF -> 10uF; footprint Capacitor_SMD:C_0805_2012Metric -> Capacitor_SMD:C_1206_3216Metric
- C4: value 68pF -> 100nF
- C5: value 22uF -> 100pF; footprint Capacitor_SMD:C_1206_3216Metric -> Capacitor_SMD:C_0805_2012Metric
- C8: value 100nF -> 10uF; footprint Capacitor_SMD:C_1206_3216Metric -> Capacitor_SMD:C_0805_2012Metric
- L2: value DR73-100-R -> DE1207-10; footprint Inductor_SMD:L_7.3x7.3_H3.5 -> Inductor_SMD:L_12x12mm_H8mm
- R1: value 182kR -> 157kR
- R2: value 18kR -> 30kR
Connections:
- net 12V: now also C3.1, U1.1 (IN), U4.2 (EN), U4.3 (IN); no longer C2.1, C7.1, C8.1
- net 3V3: now also C10.1, C11.1, U3.2 (VO)
- net 5V: now also C5.1, C6.1, C8.1, C9.1, R1.1, U3.3 (VI); no longer C10.1, C11.1
- net 9V: now also C2.1, U1.3 (OUT); no longer C4.1, C5.1, R1.1
- net GND: now also C10.2, C11.2, C3.2, C9.2, U1.2 (GND), U3.1 (GND), U4.4 (GND); no longer C6.2
- net at L2.1: now also C4.1, U4.5 (SW); no longer C9.1
- net at R1.2, R2.1: now also C5.2, U4.1 (FB); no longer C4.2
- new net: C4.2, U4.6 (BST)
- new net: C6.2, C7.1
Other:
- moved on the sheet: J1, J2, J3, J4, J5, J6, J7, J8, J9
