File: docs/PCB/Boards/RTC_Board/RTC_Board.kicad_sch (KiCad schematic)
At the start: 32 parts, among them J1 COM, Q1 BSS138-TP, Q2 BSS138-TP, Q3 AO3407A, U1 PCF8563T, U2 SIP32431DR3-T1GE3, Y1 QT3CD-32.768KEZF-T

Commit message: Boards modified.
Parts:
- R12: value 1K -> 4k7R
Changed lines of the file:
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@@
 			)
 		)
-		(property "Value" "1K"
+		(property "Value" "4k7R"
 			(at 203.2 82.55 90)
 			(effects
